File: tamagotchi.kicad_sch (KiCad schematic)
At the start: 0 parts

Commit message: make pcb
Parts:
- added BT1: Battery_Cell, Connector_PinHeader_2.54mm:PinHeader_1x02_P2.54mm_Vertical, symbol Device:Battery_Cell
- added BUZZER1: 1207-P6.5MM, easyeda2kicad:BUZ-TH_BD12.5-P6.50-D1.4, symbol easyeda2kicad:1207-P6.5MM
- added SW1, SW2, SW3: SW_Push, easyeda2kicad:SW-TH_4P-L4.5-W4.5-P3.00-LS4.8, symbol Switch:SW_Push
- added U1: XIAO-ESP32-C3-SMD, XIAO:XIAO-ESP32-C3-DIP-SMD, symbol Seeed_Studio_XIAO_Series:XIAO-ESP32-C3-SMD
- added U2: HS96L03W2C03, easyeda2kicad:OLED-TH_L27.8-W27.2-P2.54_C9900033791, symbol easyeda2kicad:HS96L03W2C03
Connections:
- new net: BUZZER1.1 (+), U1.11 (GPIO10_D10_MOSI)
- new net: SW1.2, U1.1 (GPIO2_A0_D0)
- new net: SW2.2, U1.2 (GPIO3_A1_D1)
- new net: SW3.2, U1.3 (GPIO4_A2_D2)
- new net: U1.5 (GPIO6_D4_SDA), U2.4 (SDA)
- new net: U1.6 (GPIO7_D5_SCL), U2.3 (SCL)
- new net +3V3: U1.12 (3V3), U2.2 (VCC)
- new net +5V: U1.14 (5V)
- new net +BATT: BT1.1 (+), U1.15 (BAT)
- new net GND: BT1.2 (-), BUZZER1.2 (-), SW1.1, SW2.1, SW3.1, U1.13 (GND), U2.1 (GND)
- no-connect marks 0 -> 11
